File: hardware/stmounter.kicad_pcb (KiCad board)
At the start: 2 copper layers, 1 part, among them U1 STM32F103C8Tx

Commit message: Progress
Parts:
- added C1: 22uF, Capacitor_SMD:C_0603_1608Metric, F.Cu at (176.4, 102.9)
- added C2: 22uF, Capacitor_SMD:C_0603_1608Metric, F.Cu at (164.3, 79.4)
- added FB1: 120Ω@100MHz, Inductor_SMD:L_0603_1608Metric, F.Cu at (162.0, 79.0)
- added J1: USB_C_Receptacle_USB2.0_14P, Connector_USB:USB_C_Receptacle_GCT_USB4105-xx-A_16P_TopMnt_Horizontal, F.Cu at (158.9, 72.6)
- added J2: Conn_01x20, Connector_PinSocket_2.54mm:PinSocket_1x20_P2.54mm_Vertical, F.Cu at (167.8, 119.9)
- added J3: Conn_01x20, Connector_PinSocket_2.54mm:PinSocket_1x20_P2.54mm_Vertical, F.Cu at (150.0, 119.9)
- added R1: 5.1k, Resistor_SMD:R_0402_1005Metric, F.Cu at (160.6, 78.4)
- added R2: 5.1k, Resistor_SMD:R_0402_1005Metric, F.Cu at (157.4, 78.4)
- added U2: SRV05-4, Package_TO_SOT_SMD:SOT-23-6, F.Cu at (157.1, 84.9)
- added U3: AMS1117-3.3, Package_TO_SOT_SMD:SOT-223-3_TabPin2, F.Cu at (162.4, 85.2)
- moved U1 9.66 mm to (158.9, 95.8), turned to 90 degrees
Connections:
- U1 pad 1: unconnected-(U1-VBAT-Pad1) -> +3V3
- U1 pad 23: Net-(U1-VSS-Pad23) -> GND
- U1 pad 24: unconnected-(U1-VDD-Pad24) -> +3V3
- U1 pad 3: unconnected-(U1-PC14-Pad3) -> /OSC_32_IN
- U1 pad 32: unconnected-(U1-PA11-Pad32) -> /D-
- U1 pad 33: unconnected-(U1-PA12-Pad33) -> /D+
- U1 pad 34: unconnected-(U1-PA13-Pad34) -> /GPIO0
- U1 pad 35: Net-(U1-VSS-Pad23) -> GND
- U1 pad 36: unconnected-(U1-VDD-Pad36) -> +3V3
- U1 pad 37: unconnected-(U1-PA14-Pad37) -> /GPIO1
- U1 pad 38: unconnected-(U1-PA15-Pad38) -> /GPIO2
- U1 pad 39: unconnected-(U1-PB3-Pad39) -> /GPIO3
- U1 pad 4: unconnected-(U1-PC15-Pad4) -> /OSC_32_OUT
- U1 pad 40: unconnected-(U1-PB4-Pad40) -> /GPIO4
- U1 pad 41: unconnected-(U1-PB5-Pad41) -> /GPIO5
- U1 pad 42: unconnected-(U1-PB6-Pad42) -> /GPIO6
- U1 pad 43: unconnected-(U1-PB7-Pad43) -> /GPIO7
- U1 pad 47: Net-(U1-VSS-Pad23) -> GND
- U1 pad 48: unconnected-(U1-VDD-Pad48) -> +3V3
- U1 pad 7: unconnected-(U1-NRST-Pad7) -> Net-(U1-NRST)
- U1 pad 8: unconnected-(U1-VSSA-Pad8) -> GND
- U1 pad 9: unconnected-(U1-VDDA-Pad9) -> +3V3
Routing:
- net /GPIO0: track 0.00 -> 22.9 mm
- net /GPIO1: track 0.00 -> 21.1 mm
- net +5V: track 0.00 -> 18.6 mm, vias 0 -> 2
- net VBUS: track 0.00 -> 18.0 mm
- net /D-: track 0.00 -> 16.8 mm
- net /D+: track 0.00 -> 16.8 mm
- net /GPIO2: track 0.00 -> 16.7 mm
- net /GPIO3: track 0.00 -> 14.8 mm
- net /GPIO4: track 0.00 -> 12.9 mm
- net /GPIO5: track 0.00 -> 11.0 mm
- net /GPIO6: track 0.00 -> 6.49 mm
- net /GPIO29: track 0.00 -> 5.82 mm
- net /GPIO7: track 0.00 -> 5.36 mm
- net Net-(J1-CC2): track 0.00 -> 1.67 mm
- net Net-(J1-CC1): track 0.00 -> 1.63 mm
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- added copper zone on B.Cu, net GND
- added copper zone on F.Cu, net GND
Other:
- board outline added: 21 x 51 mm

Commit message: Progress
Parts:
- added C10: 10pF, Capacitor_SMD:C_0402_1005Metric, F.Cu at (160.2, 107.0)
- added C11: 10pF, Capacitor_SMD:C_0402_1005Metric, F.Cu at (162.8, 104.8)
- added C12: 15pF, Capacitor_SMD:C_0402_1005Metric, F.Cu at (156.9, 105.7)
- added C13: 15pF, Capacitor_SMD:C_0402_1005Metric, F.Cu at (155.1, 105.7)
- added C3: 100nF, Capacitor_SMD:C_0402_1005Metric, F.Cu at (156.1, 90.2)
- added C4: 100nF, Capacitor_SMD:C_0402_1005Metric, F.Cu at (154.2, 99.5)
- added C5: 100nF, Capacitor_SMD:C_0402_1005Metric, F.Cu at (155.2, 100.9)
- added C6: 100nF, Capacitor_SMD:C_0402_1005Metric, F.Cu at (160.2, 101.5)
- added C7: 100nF, Capacitor_SMD:C_0402_1005Metric, F.Cu at (163.6, 92.2)
- added C8: 10uF, Capacitor_SMD:C_0402_1005Metric, F.Cu at (160.2, 102.4)
- added C9: 1uF, Capacitor_SMD:C_0402_1005Metric, F.Cu at (154.2, 100.9)
- added R4: 0, Resistor_SMD:R_0402_1005Metric, F.Cu at (158.8, 101.9)
- added R5: 390, Resistor_SMD:R_0402_1005Metric, F.Cu at (157.5, 101.9)
- added Y1: 16MHz 9pF, Crystal:Crystal_SMD_3225-4Pin_3.2x2.5mm, F.Cu at (160.2, 104.8)
- added Y2: 32.768kHz 12.5pF, Crystal:Crystal_SMD_3215-2Pin_3.2x1.5mm, F.Cu at (156.0, 104.0)
- moved C1 17.7 mm to (163.9, 90.3)
- moved C2 0.80 mm to (163.5, 79.2), turned to -90 degrees
Connections:
- J1 pad S1: GND -> unconnected-(J1-SHIELD-PadS1)
- U1 pad 10: unconnected-(U1-PA0-Pad10) -> /GPIO18
- U1 pad 11: unconnected-(U1-PA1-Pad11) -> /GPIO16
- U1 pad 12: unconnected-(U1-PA2-Pad12) -> /GPIO17
- U1 pad 13: unconnected-(U1-PA3-Pad13) -> /GPIO19
- U1 pad 14: unconnected-(U1-PA4-Pad14) -> /GPIO20
- U1 pad 15: unconnected-(U1-PA5-Pad15) -> /GPIO21
- U1 pad 16: unconnected-(U1-PA6-Pad16) -> /GPIO22
- U1 pad 17: unconnected-(U1-PA7-Pad17) -> /GPIO23
- U1 pad 18: unconnected-(U1-PB0-Pad18) -> /GPIO24
- U1 pad 19: unconnected-(U1-PB1-Pad19) -> /GPIO25
- U1 pad 20: unconnected-(U1-PB2-Pad20) -> /GPIO26
- U1 pad 21: unconnected-(U1-PB10-Pad21) -> /GPIO27
- U1 pad 22: unconnected-(U1-PB11-Pad22) -> /GPIO28
- U1 pad 25: unconnected-(U1-PB12-Pad25) -> /GPIO29
- U1 pad 5: unconnected-(U1-PD0-Pad5) -> /OSC_IN
- U1 pad 6: unconnected-(U1-PD1-Pad6) -> /OSC_OUT
Routing:
- net /GPIO16: track 0.00 -> 23.5 mm
- net /GPIO17: track 0.00 -> 20.4 mm
- net /GPIO18: track 0.00 -> 18.2 mm
- net /GPIO19: track 0.00 -> 13.7 mm
- net /GPIO28: track 0.00 -> 13.6 mm
- net /GPIO27: track 0.00 -> 12.8 mm
- net /GPIO20: track 0.00 -> 11.7 mm
- net /GPIO29: track 5.82 -> 16.9 mm
- net /GPIO26: track 0.00 -> 11.0 mm
- net +3V3: track 0.00 -> 9.89 mm, vias 0 -> 2
- net /GPIO21: track 0.00 -> 9.83 mm
- net GND: track 0.00 -> 8.46 mm, vias 10 -> 32
- net /OSC_IN: track 0.00 -> 7.58 mm
- net /OSC_32_IN: track 0.00 -> 6.73 mm
- net /GPIO25: track 0.00 -> 6.57 mm
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- added copper zone on F.Cu, net +3V3

Commit message: Progress
Parts:
- removed U1: STM32F103C8Tx, Package_QFP:LQFP-48_7x7mm_P0.5mm
- added C14: 100nF, Capacitor_SMD:C_0402_1005Metric, F.Cu at (163.6, 106.9)
- added R3: 1.5k, Resistor_SMD:R_0402_1005Metric, F.Cu at (156.3, 88.2)
- added R8: 10k, Resistor_SMD:R_0402_1005Metric, F.Cu at (154.1, 110.8)
- added SW1: SW_Push, stmounter:TS-1088-AR02016-Switch-SMD, F.Cu at (155.9, 115.8)
- added SW2: SW_Push, stmounter:TS-1088-AR02016-Switch-SMD, F.Cu at (161.9, 115.8)
- added U5: STM32F373CCTx, Package_QFP:LQFP-48_7x7mm_P0.5mm, F.Cu at (158.9, 95.8)
- C10, C11: value 10pF -> 15pF
- R5: value 390 -> 470
- Y1: value 16MHz 9pF -> 25MHz 12pF
- Y2: value 32.768kHz 12.5pF -> 32kHz 12.5pF
- moved R1 2.19 mm to (162.8, 78.3), turned to 180 degrees
- moved C2 1.94 mm to (165.2, 78.4)
- moved FB1 1.69 mm to (160.4, 78.5), turned to 180 degrees
- moved U2 1.43 mm to (156.1, 83.9), turned to 90 degrees
- moved U3 1.31 mm to (161.4, 84.4)
- moved C1 1.29 mm to (162.9, 89.6)
- moved R2 1.27 mm to (156.1, 78.3), turned to 0 degrees
- moved J1 0.41 mm to (158.9, 73.0)
- moved Y2 0.10 mm to (156.1, 104.0)
- moved R5 0.05 mm to (157.6, 101.9)
Connections:
- J1 pad S1: unconnected-(J1-SHIELD-PadS1) -> GND
- U2 pad 1: /D- -> /D+
- U2 pad 3: /D+ -> /D-
- U2 pad 4: /D+ -> /D-
- U2 pad 6: /D- -> /D+
Routing:
- net +3V3: track 9.89 -> 66.8 mm, vias 2 -> 9
- net /GPIO15: track 0.00 -> 24.9 mm
- net /GPIO14: track 0.00 -> 22.9 mm
- net Net-(U5-NRST): track 0.00 -> 21.5 mm, vias 0 -> 2
- net /BOOTSEL: track 0.00 -> 20.2 mm, vias 0 -> 2
- net /GPIO13: track 0.00 -> 19.4 mm
- net /GPIO12: track 0.00 -> 17.4 mm
- net VBUS: track 18.0 -> 1.86 mm
- net /GPIO9: track 0.00 -> 15.9 mm, vias 0 -> 1
- net /GPIO11: track 0.00 -> 15.5 mm
- net /GPIO10: track 0.00 -> 13.6 mm
- net /GPIO8: track 0.00 -> 13.5 mm, vias 0 -> 1
- net /GPIO5: track 11.0 -> 0.00 mm
- net /GPIO7: track 5.36 -> 12.3 mm, vias 0 -> 1
- net /GPIO22: track 5.79 -> 0.00 mm
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- added copper zone on F.Cu, net VBUS
Other:
- outline, holes or cut-outs redrawn
- board text added: "BOOT"
- board text added: "RESET"

Commit message: Progress
Parts:
- removed C8: 10uF, Capacitor_SMD:C_0402_1005Metric
- added D1: WHITE, LED_SMD:LED_0603_1608Metric, F.Cu at (161.7, 109.5)
- added D2: WHITE, LED_SMD:LED_0603_1608Metric, F.Cu at (156.7, 109.5)
- added R6: 680, Resistor_SMD:R_0402_1005Metric, F.Cu at (154.7, 108.8)
- added R7: 680, Resistor_SMD:R_0402_1005Metric, F.Cu at (164.3, 100.4)
- moved C3 10.9 mm to (165.0, 96.5)
- moved C14 4.01 mm to (163.3, 110.9)
- moved C9 1.62 mm to (155.7, 101.4), turned to 180 degrees
- moved C5 1.55 mm to (155.7, 102.4), turned to 180 degrees
- moved R3 1.23 mm to (157.0, 89.2)
- moved R8 0.43 mm to (153.7, 110.7)
- moved C6 0.25 mm to (160.4, 101.5)
- moved C1 0.06 mm to (162.9, 89.5)
Connections:
- J2 pad 15: /GPIO27 -> /ADC_VREF
- J2 pad 16: /GPIO28 -> +3V3
- J2 pad 17: /GPIO29 -> +3V3
- U5 pad 10: unconnected-(U5-PA0-Pad10) -> /LED1
- U5 pad 11: unconnected-(U5-PA1-Pad11) -> /GPIO16
- U5 pad 12: unconnected-(U5-PA2-Pad12) -> /GPIO17
- U5 pad 13: unconnected-(U5-PA3-Pad13) -> /GPIO18
- U5 pad 14: unconnected-(U5-PA4-Pad14) -> /GPIO19
- U5 pad 15: unconnected-(U5-PA5-Pad15) -> /GPIO20
- U5 pad 16: unconnected-(U5-PA6-Pad16) -> /GPIO21
- U5 pad 18: unconnected-(U5-PB0-Pad18) -> /GPIO22
- U5 pad 19: unconnected-(U5-PB1-Pad19) -> /GPIO23
- U5 pad 2: unconnected-(U5-PC13-Pad2) -> /GPIO15
- U5 pad 20: unconnected-(U5-PB2-Pad20) -> /GPIO24
- U5 pad 21: unconnected-(U5-PE8-Pad21) -> /GPIO25
- U5 pad 22: unconnected-(U5-PE9-Pad22) -> /GPIO26
- U5 pad 25: unconnected-(U5-VREFSD+-Pad25) -> /ADC_VREF
- U5 pad 26: unconnected-(U5-PB14-Pad26) -> /GPIO29
- U5 pad 27: unconnected-(U5-PB15-Pad27) -> /GPIO28
- U5 pad 28: unconnected-(U5-PD8-Pad28) -> /LED2
- U5 pad 29: unconnected-(U5-PA8-Pad29) -> /GPIO9
- U5 pad 30: unconnected-(U5-PA9-Pad30) -> /GPIO4
- U5 pad 31: unconnected-(U5-PA10-Pad31) -> /GPIO3
- U5 pad 34: unconnected-(U5-PA13-Pad34) -> /GPIO0
- U5 pad 35: unconnected-(U5-PF6-Pad35) -> /GPIO1
- U5 pad 36: unconnected-(U5-PF7-Pad36) -> /GPIO2
- U5 pad 37: unconnected-(U5-PA14-Pad37) -> /GPIO5
- U5 pad 38: unconnected-(U5-PA15-Pad38) -> /GPIO6
- U5 pad 39: unconnected-(U5-PB3-Pad39) -> /GPIO7
- U5 pad 40: unconnected-(U5-PB4-Pad40) -> /GPIO8
- U5 pad 41: unconnected-(U5-PB5-Pad41) -> /GPIO10
- U5 pad 42: unconnected-(U5-PB6-Pad42) -> /GPIO11
- U5 pad 43: unconnected-(U5-PB7-Pad43) -> /GPIO12
- U5 pad 45: unconnected-(U5-PB8-Pad45) -> /GPIO13
- U5 pad 46: unconnected-(U5-PB9-Pad46) -> /GPIO14
Routing:
- net /LED2: track 0.00 -> 23.9 mm, vias 0 -> 2
- net /GPIO29: track 16.7 -> 0.00 mm
- net /GPIO28: track 14.9 -> 0.00 mm
- net /GPIO27: track 12.8 -> 0.00 mm
- net /ADC_VREF: track 0.00 -> 11.3 mm
- net Net-(D1-A): track 0.00 -> 10.1 mm, vias 0 -> 2
- net /GPIO5: track 0.00 -> 8.52 mm
- net /GPIO8: track 13.5 -> 5.77 mm, vias 1 -> 0
- net /GPIO7: track 12.3 -> 4.93 mm, vias 1 -> 0
- net +3V3: track 66.8 -> 74.2 mm
- net /GPIO22: track 0.00 -> 7.34 mm
- net /GPIO6: track 12.0 -> 5.37 mm, vias 1 -> 0
- net /GPIO1: track 25.6 -> 20.2 mm
- net /LED1: track 0.00 -> 4.58 mm
- net /GPIO15: track 24.9 -> 29.4 mm
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Other:
- board text added: "3V3"
- board text added: "5V"
- board text added: "GND"
- board text added: "PA1"
- board text added: "PA10"
- board text added: "PA13"
- board text added: "PA14"
- board text added: "PA15"
- board text added: "PA2"
- board text added: "PA3"
- board text added: "PA4"
- board text added: "PA5"
- board text added: "PA6"
- board text added: "PA8"
- board text added: "PA9"
- board text added: "PB0"
- board text added: "PB1"
- board text added: "PB2"
- board text added: "PB3"
- board text added: "PB4"
- board text added: "PB5"
- board text added: "PB6"
- board text added: "PB7"
- board text added: "PB8"
- board text added: "PB9"
- board text added: "PC13"
- board text added: "PE8"
- board text added: "PE9"
- board text added: "PF6"
- board text added: "PF7"
- board text added: "VBUS"
- board text added: "VREF"
