File: hardware/stmounter.kicad_sch (KiCad schematic)
At the start: 2 parts, among them J1 USB_C_Receptacle_USB2.0_14P, U1 STM32F103C8Tx

Commit message: Progress
Parts:
- added C1, C2: 22uF, Capacitor_SMD:C_0603_1608Metric, symbol Device:C
- added FB1: 120Ω@100MHz, Inductor_SMD:L_0603_1608Metric, symbol Device:FerriteBead
- added J2, J3: Conn_01x20, Connector_PinSocket_2.54mm:PinSocket_1x20_P2.54mm_Vertical, symbol Connector_Generic:Conn_01x20
- added R1, R2: 5.1k, Resistor_SMD:R_0402_1005Metric, symbol Device:R
- added R3: 1.5k, symbol Device:R
- added SW1: SW_Push, symbol Switch:SW_Push
- added U2: SRV05-4, Package_TO_SOT_SMD:SOT-23-6, symbol Power_Protection:SRV05-4
- added U3: AMS1117-3.3, Package_TO_SOT_SMD:SOT-223-3_TabPin2, symbol Regulator_Linear:AMS1117-3.3
- J1: footprint (none) -> Connector_USB:USB_C_Receptacle_GCT_USB4105-xx-A_16P_TopMnt_Horizontal; LCSC Part # (none) -> C2765186
Connections:
- net +3V3: now reaches U1.1 (VBAT)
- net +3V3: now also U1.24 (VDD), U1.36 (VDD), U1.48 (VDD), U1.9 (VDDA), C1.1, R3.1, U3.2 (VO)
- net GND: now reaches U1.23 (VSS), U1.35 (VSS), U1.47 (VSS)
- net GND: now also J1.A1 (GND), J1.A12 (GND), J1.B1 (GND), J1.B12 (GND), J1.S1 (SHIELD), U1.8 (VSSA), C1.2, C2.2, J2.13 (Pin_13), J2.18 (Pin_18), J2.3 (Pin_3), J2.8 (Pin_8), J3.13 (Pin_13), J3.18 (Pin_18), J3.3 (Pin_3), J3.8 (Pin_8), R1.2, R2.1, U2.2 (VN), U3.1 (GND)
- net OSC_32_IN: now reaches U1.3 (PC14)
- net D-: now reaches U1.32 (PA11)
- net D-: now also J1.A7 (D-), J1.B7 (D-), U2.1 (IO1), U2.6 (IO4)
- net D+: now reaches U1.33 (PA12)
- net D+: now also J1.A6 (D+), J1.B6 (D+), R3.2, U2.3 (IO2), U2.4 (IO3)
- net GPIO0: now reaches U1.34 (PA13)
- net GPIO0: now also J3.20 (Pin_20)
- net GPIO1: now reaches U1.37 (PA14)
- net GPIO1: now also J3.19 (Pin_19)
- net GPIO2: now reaches U1.38 (PA15)
- net GPIO2: now also J3.17 (Pin_17)
- net GPIO3: now reaches U1.39 (PB3)
- net GPIO3: now also J3.16 (Pin_16)
- net OSC_32_OUT: now reaches U1.4 (PC15)
- net GPIO4: now reaches U1.40 (PB4)
- net GPIO4: now also J3.15 (Pin_15)
- net GPIO5: now reaches U1.41 (PB5)
- net GPIO5: now also J3.14 (Pin_14)
- net GPIO6: now reaches U1.42 (PB6)
- net GPIO6: now also J3.12 (Pin_12)
- net GPIO7: now reaches U1.43 (PB7)
- net GPIO7: now also J3.11 (Pin_11)
- net at U1.7 (NRST): now also SW1.2
- net VBUS: now reaches J1.A4 (VBUS), J1.A9 (VBUS), J1.B4 (VBUS), J1.B9 (VBUS)
- net VBUS: now also FB1.1, J2.20 (Pin_20)
- net at J1.A5 (CC1): now also R1.1
- net at J1.B5 (CC2): now also R2.2
- new net +5V: C2.1, FB1.2, J2.19 (Pin_19), U2.5 (VP), U3.3 (VI)
- new net GPIO10: J3.7 (Pin_7)
- new net GPIO11: J3.6 (Pin_6)
- new net GPIO12: J3.5 (Pin_5)
- new net GPIO13: J3.4 (Pin_4)
- new net GPIO14: J3.2 (Pin_2)
- new net GPIO15: J3.1 (Pin_1)
- new net GPIO16: J2.1 (Pin_1)
- new net GPIO17: J2.2 (Pin_2)
- new net GPIO18: J2.4 (Pin_4)
- new net GPIO19: J2.5 (Pin_5)
- new net GPIO20: J2.6 (Pin_6)
- new net GPIO21: J2.7 (Pin_7)
- new net GPIO22: J2.9 (Pin_9)
- new net GPIO23: J2.10 (Pin_10)
- new net GPIO24: J2.11 (Pin_11)
- new net GPIO25: J2.12 (Pin_12)
- new net GPIO26: J2.14 (Pin_14)
- new net GPIO27: J2.15 (Pin_15)
- new net GPIO28: J2.16 (Pin_16)
- new net GPIO29: J2.17 (Pin_17)
- new net GPIO8: J3.10 (Pin_10)
- new net GPIO9: J3.9 (Pin_9)
Other:
- note added: "Pullup needed by stm32"
- note removed: "USB DP -> 1.5k pullup to 3.3v"
- moved on the sheet: U1

Commit message: Progress
Parts:
- added C10, C11: 10pF, Capacitor_SMD:C_0402_1005Metric, symbol Device:C
- added C12, C13: 15pF, Capacitor_SMD:C_0402_1005Metric, symbol Device:C
- added C3, C4, C5, C6, C7: 100nF, Capacitor_SMD:C_0402_1005Metric, symbol Device:C
- added C8: 10uF, Capacitor_SMD:C_0402_1005Metric, symbol Device:C
- added C9: 1uF, Capacitor_SMD:C_0402_1005Metric, symbol Device:C
- added R4: 0, Resistor_SMD:R_0402_1005Metric, symbol Device:R
- added R5: 390, Resistor_SMD:R_0402_1005Metric, symbol Device:R
- added Y1: 16MHz 9pF, Crystal:Crystal_SMD_3225-4Pin_3.2x2.5mm, symbol Device:Crystal_GND24
- added Y2: 32.768kHz 12.5pF, Crystal:Crystal_SMD_3215-2Pin_3.2x1.5mm, symbol Device:Crystal
Connections:
- net +3V3: now also C3.1, C4.1, C5.1, C6.1, C7.1, C8.1, C9.1
- net GND: now also C10.1, C11.1, C12.1, C13.1, C3.2, C4.2, C5.2, C6.2, C7.2, C8.2, C9.2, Y1.2, Y1.4; no longer J1.S1 (SHIELD)
- net GPIO16: now also U1.11 (PA1)
- net GPIO17: now also U1.12 (PA2)
- net GPIO18: now also U1.10 (PA0)
- net GPIO19: now also U1.13 (PA3)
- net GPIO20: now also U1.14 (PA4)
- net GPIO21: now also U1.15 (PA5)
- net GPIO22: now also U1.16 (PA6)
- net GPIO23: now also U1.17 (PA7)
- net GPIO24: now also U1.18 (PB0)
- net GPIO25: now also U1.19 (PB1)
- net GPIO26: now also U1.20 (PB2)
- net GPIO27: now also U1.21 (PB10)
- net GPIO28: now also U1.22 (PB11)
- net GPIO29: now also U1.25 (PB12)
- net OSC_32_IN: now also C13.2, Y2.1
- net OSC_32_OUT: now also R5.2
- net OSC_IN: now reaches U1.5 (PD0)
- net OSC_IN: now also C10.2, Y1.3
- net OSC_OUT: now reaches U1.6 (PD1)
- net OSC_OUT: now also R4.2
- new net: C11.2, R4.1, Y1.1
- new net: C12.2, R5.1, Y2.2
Other:
- moved on the sheet: C1, C2, FB1, J1, J2, J3, R1, R2, R3, SW1, U1, U2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

Commit message: Progress
Parts:
- removed U1: STM32F103C8Tx, Package_QFP:LQFP-48_7x7mm_P0.5mm, symbol MCU_ST_STM32F1:STM32F103C8Tx
- added C14: 100nF, Capacitor_SMD:C_0402_1005Metric, symbol Device:C
- added R8: 10k, Resistor_SMD:R_0402_1005Metric, symbol Device:R
- added SW2: SW_Push, stmounter:TS-1088-AR02016-Switch-SMD, symbol Switch:SW_Push
- added U5: STM32F373CCTx, Package_QFP:LQFP-48_7x7mm_P0.5mm, symbol MCU_ST_STM32F3:STM32F373CCTx
- C1, C2: LCSC Part # (none) -> C59461
- C10, C11: value 10pF -> 15pF; LCSC Part # (none) -> C1548
- C12, C13: LCSC Part # (none) -> C1548
- C3, C4, C5, C6, C7: LCSC Part # (none) -> C1525
- C8: LCSC Part # (none) -> C15525
- C9: LCSC Part # (none) -> C52923
- R1, R2: LCSC Part # (none) -> C25905
- R3: footprint (none) -> Resistor_SMD:R_0402_1005Metric; LCSC Part # (none) -> C25867
- R4: LCSC Part # (none) -> C17168
- R5: value 390 -> 470; LCSC Part # (none) -> C25117
- SW1: footprint (none) -> stmounter:TS-1088-AR02016-Switch-SMD; LCSC Part # (none) -> C720477
- Y1: value 16MHz 9pF -> 25MHz 12pF; LCSC Part # C13738 -> C9006
- Y2: value 32.768kHz 12.5pF -> 32kHz 12.5pF; LCSC Part # (none) -> C32346 (
Connections:
- net +3V3: now also SW1.1, U5.1 (VBAT), U5.17 (VDD), U5.24 (VDDSD), U5.48 (VDD), U5.9 (VDDA)
- net D+: now also U2.1 (IO1), U2.6 (IO4), U5.33 (PA12); no longer U2.3 (IO2), U2.4 (IO3)
- net D-: now also U2.3 (IO2), U2.4 (IO3), U5.32 (PA11); no longer U2.1 (IO1), U2.6 (IO4)
- net GND: now also J1.S1 (SHIELD), C14.2, R8.1, SW2.1, U5.23 (VSSSD), U5.47 (VSS), U5.8 (VSSA)
- net OSC_32_IN: now also U5.3 (PC14)
- net OSC_32_OUT: now also U5.4 (PC15)
- net OSC_IN: now also U5.5 (PF0)
- net OSC_OUT: now also U5.6 (PF1)
- net BOOTSEL: now reaches SW1.2
- net BOOTSEL: now also R8.2, U5.44 (BOOT0)
- new net: C14.1, SW2.2, U5.7 (NRST)
Other:
- note added: "D+"
- note added: "D-"
- note added: "OSC32_IN"
- note added: "OSC32_OUT"
- note added: "OSC_IN"
- note added: "OSC_OUT"
- note added: "SWCLK"
- note added: "SWDIO"
- moved on the sheet: C10, C11, C12, C13, C3, C4, C5, C6, C7, C8, C9, R3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

Commit message: Progress
Parts:
- removed C8: 10uF, Capacitor_SMD:C_0402_1005Metric, symbol Device:C
- added D1, D2: WHITE, LED_SMD:LED_0603_1608Metric, symbol Device:LED
- added R6, R7: 680, Resistor_SMD:R_0402_1005Metric, symbol Device:R
Connections:
- net GPIO27 is gone; now on net ADC_VREF: J2.15 (Pin_15)
- net +3V3: now also J2.16 (Pin_16), J2.17 (Pin_17)
- net GND: now also D1.1 (K), D2.1 (K)
- net GPIO0: now also U5.34 (PA13)
- net GPIO1: now also U5.35 (PF6)
- net GPIO10: now also U5.41 (PB5)
- net GPIO11: now also U5.42 (PB6)
- net GPIO12: now also U5.43 (PB7)
- net GPIO13: now also U5.45 (PB8)
- net GPIO14: now also U5.46 (PB9)
- net GPIO15: now also U5.2 (PC13)
- net GPIO16: now also U5.11 (PA1)
- net GPIO17: now also U5.12 (PA2)
- net GPIO18: now also U5.13 (PA3)
- net GPIO19: now also U5.14 (PA4)
- net GPIO2: now also U5.36 (PF7)
- net GPIO20: now also U5.15 (PA5)
- net GPIO21: now also U5.16 (PA6)
- net GPIO22: now also U5.18 (PB0)
- net GPIO23: now also U5.19 (PB1)
- net GPIO24: now also U5.20 (PB2)
- net GPIO25: now also U5.21 (PE8)
- net GPIO26: now also U5.22 (PE9)
- net GPIO28: now also U5.27 (PB15); no longer J2.16 (Pin_16)
- net GPIO29: now also U5.26 (PB14); no longer J2.17 (Pin_17)
- net GPIO3: now also U5.31 (PA10)
- net GPIO4: now also U5.30 (PA9)
- net GPIO5: now also U5.37 (PA14)
- net GPIO6: now also U5.38 (PA15)
- net GPIO7: now also U5.39 (PB3)
- net GPIO8: now also U5.40 (PB4)
- net GPIO9: now also U5.29 (PA8)
- net LED1: now reaches U5.10 (PA0)
- net LED1: now also R7.1
- net ADC_VREF: now reaches U5.25 (VREFSD+)
- net LED2: now reaches U5.28 (PD8)
- net LED2: now also R6.1
- new net: D1.2 (A), R7.2
- new net: D2.2 (A), R6.2
Other:
- note added: "MISO1"
- note added: "MISO3/TX2"
- note added: "MOSI1"
- note added: "MOSI3/RX2"
- note added: "SCK1"
- note added: "SCK3"
- moved on the sheet: C1, C10, C11, C12, C13, C14, C2, C4, C5, C6, C7, C9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
